Commit message: fix rviz

File: src/rover_description/robots/rover.urdf.xacro (robot description, xacro)
@@ -9,5 +9,5 @@
   <link name="base_footprint"/>
   <xacro:base_v0 parent="base_footprint">
-	<origin xyz="0 0 0.3"/>
+	<origin xyz="0 0 0.3" rpy="0 0 -1.570796"/>
   </xacro:base_v0>
   <!-- Suspension -->

Commit message: add updated model

File: src/rover_description/robots/rover.urdf.xacro (robot description, xacro)
@@ -9,25 +9,25 @@
   <link name="base_footprint"/>
   <xacro:base_v0 parent="base_footprint">
-	<origin xyz="0 0 0.3" rpy="0 0 -1.570796"/>
+	<origin xyz="0 0 0.25" rpy="0 0 -1.570796"/>
   </xacro:base_v0>
   <!-- Suspension -->
   <!-- Front Right Sus -->
   <xacro:steering_v0 prefix="front_right" parent="base_link">
-	<origin xyz="0.26937 0.30011 -0.14453" rpy="0 0 0.15"/>
+	<origin xyz="0.63104 -0.25952 -0.0205" rpy="0 0 0"/>
 	<axis xyz="0 0 1"/>
   </xacro:steering_v0>
   <!-- Front Left Sus -->
   <xacro:steering_v0 prefix="front_left" parent="base_link">
-	<origin xyz="-0.26927 0.30019 -0.14943" rpy="0 0 ${M_PI+0.15}"/>
+	<origin xyz="0.63104 0.25952 -0.0205" rpy="0 0 ${M_PI}"/>
 	<axis xyz="0 0 1"/>
   </xacro:steering_v0>
   <!-- Rear Right Sus -->
   <xacro:steering_v0 prefix="rear_right" parent="base_link">
-	<origin xyz="0.26948 -0.2789 -0.15361" rpy="0 0 0.15"/>
+	<origin xyz="-0.63104 -0.25952 -0.0205" rpy="0 0 0"/>
 	<axis xyz="0 0 1"/>
   </xacro:steering_v0>
   <!-- Rear Left Sus -->
   <xacro:steering_v0 prefix="rear_left" parent="base_link">
-	<origin xyz="-0.26951 -0.27994 -0.15131" rpy="0 0 ${M_PI+0.15}"/>
+	<origin xyz="-0.63104 0.25952 -0.0205" rpy="0 0 ${M_PI}"/>
 	<axis xyz="0 0 1"/>
   </xacro:steering_v0>
@@ -35,21 +35,21 @@
   <!-- Front Right Wheel -->
   <xacro:wheel_v0 prefix="ffr" parent="front_right_steering_link">
-	<origin xyz="0.00049811 -4.3395E-05 -0.085" rpy="0 0 0"/>
-	<axis xyz="-1 0.1 0"/>
+	<origin xyz="0 0 -0.129" rpy="0 0 0"/>
+	<axis xyz="0 -1 0"/>
   </xacro:wheel_v0>
   <!--  Front Left Wheel -->
   <xacro:wheel_v0 prefix="ffl" parent="front_left_steering_link">
-	<origin xyz="0.007 0 -0.085" rpy="0 0 ${M_PI}"/>
-	<axis xyz="-1 0.1 0"/>
+	<origin xyz="0 0 -0.129" rpy="0 0 0"/>
+	<axis xyz="0 -1 0"/>
   </xacro:wheel_v0>
   <!-- Rear Right Wheel -->
   <xacro:wheel_v0 prefix="rfr" parent="rear_right_steering_link">
-	<origin xyz="0.0004994 -2.4447E-05 -0.085" rpy="0 0 0"/>
-	<axis xyz="-1 0.1 0"/>
+	<origin xyz="0 0 -0.129" rpy="0 0 0"/>
+	<axis xyz="0 -1 0"/>
   </xacro:wheel_v0>
   <!--  Rear Left Wheel -->
   <xacro:wheel_v0 prefix="rfl" parent="rear_left_steering_link">
-	<origin xyz="0.0069992 0.00010415 -0.085" rpy="0 0 ${M_PI}"/>
-	<axis xyz="-1 0.1 0"/>
+	<origin xyz="0 0 -0.129" rpy="0 0 0"/>
+	<axis xyz="0 -1 0"/>
   </xacro:wheel_v0>
   <!-- ===============  Wheel Transmission =============== -->

File: src/rover_description/urdf/base/base.gazebo.xacro (robot description, xacro)
@@ -6,4 +6,5 @@
       <mu1 value="0.05" />
       <mu2 value="0.05" />
+      <material>Gazebo/Black</material>
     </gazebo>
   </xacro:macro>

File: src/rover_description/urdf/base/base.urdf.xacro (robot description, xacro)
@@ -10,31 +10,34 @@
 	<link name="base_link">
 	  <visual>
-		<geometry>
-		  <mesh filename="package://rover_description/meshes/STL/base/base_link.stl"/>
-		</geometry>
+	    <origin
+		  xyz="0 0 0"
+		  rpy="0 0 0" />
+	    <geometry>
+		  <mesh filename="package://rover_description/meshes/STL/base/base_link.STL"/>
+	    </geometry>
 	  </visual>
-	<collision>
-      <origin
-        xyz="0.0090992 -0.050658 -0.002"
-        rpy="0 0 0" />
-      <geometry>
-        <mesh
-          filename="package://rover_description/meshes/STL/base/base_link.stl" />
-      </geometry>
-    </collision>
-		<inertial>
+	  <collision>
+	    <origin
+		  xyz="0 0 0"
+		  rpy="0 0 0" />
+	    <geometry>
+		  <mesh
+		  filename="package://rover_description/meshes/STL/base/base_link.STL" />
+	    </geometry>
+	  </collision>
+	  <inertial>
 		<origin
-			xyz="0 0 0"
+			xyz="-0.00062726 0.00031624 0.021725"
 			rpy="0 0 0" />
 		<mass
-			value="8.0206" />
-		<inertia
-			ixx="0.0159"
-			ixy="7.4996E-05"
-			ixz="-8.6149E-05"
-			iyy="0.011714"
-			iyz="0.0007604"
-			izz="0.015363" />
-		</inertial>
+			value="4.6623" />
+	    <inertia
+			ixx="0.021722"
+			ixy="6.1565E-06"
+			ixz="2.5518E-06"
+			iyy="0.08573"
+			iyz="6.3788E-07"
+			izz="0.10519" />
+	  </inertial>
 	</link>
   </xacro:macro>

File: src/rover_description/urdf/suspension/suspension.gazebo.xacro (robot description, xacro)
@@ -6,4 +6,5 @@
       <mu1 value="0.05" />
       <mu2 value="0.05" />
+    <material>Gazebo/Blue</material>
     </gazebo>
   </xacro:macro>

File: src/rover_description/urdf/suspension/suspension.urdf.xacro (robot description, xacro)
@@ -14,15 +14,15 @@
 	  <inertial>
       <origin
-        xyz="-0.044924 0.0039137 -0.040662"
+        xyz="0.00015592 -0.03241 -0.074114"
         rpy="0 0 0" />
       <mass
-        value="0.23292" />
+        value="0.26619" />
       <inertia
-        ixx="7.0788E-05"
-        ixy="1.2054E-05"
-        ixz="-5.2515E-06"
-        iyy="0.00019796"
-        iyz="2.6886E-06"
-        izz="0.00017873" />
+        ixx="0.00044783"
+        ixy="1.7606E-07"
+        ixz="-1.0156E-06"
+        iyy="0.00042274"
+        iyz="-4.3434E-06"
+        izz="8.5179E-05" />
     </inertial>
     <visual>
@@ -32,5 +32,5 @@
       <geometry>
         <mesh
-          filename="package://rover_description/meshes/STL/suspension/sus_link.stl" />
+          filename="package://rover_description/meshes/STL/suspension/steering.STL" />
       </geometry>
       <material
@@ -46,5 +46,5 @@
       <geometry>
         <mesh
-          filename="package://rover_description/meshes/STL/suspension/sus_link.stl" />
+          filename="package://rover_description/meshes/STL/suspension/steering.STL" />
       </geometry>
     </collision>

File: src/rover_description/urdf/wheel/wheel.gazebo.xacro (robot description, xacro)
@@ -2,8 +2,9 @@
 <robot xmlns:xacro="http://ros.org/wiki/xacro">
   <xacro:macro name="wheel_gazebo_v0" params="prefix">
-    <gazebo reference="${prefix}_wheel_link">
-      <selfCollide>false</selfCollide>
+  <gazebo reference="${prefix}_wheel_link">
+    <selfCollide>false</selfCollide>
       <mu1 value="1.2" />
       <mu2 value="1.2" />
+      <material>Gazebo/Black</material>
     </gazebo>
   </xacro:macro>

File: src/rover_description/urdf/wheel/wheel.urdf.xacro (robot description, xacro)
@@ -14,15 +14,15 @@
 	  <inertial>
       <origin
-        xyz="0.0019728 -0.00016049 2.625E-06"
+        xyz="5.9053E-07 -0.0064734 -1.1775E-07"
         rpy="0 0 0" />
       <mass
-        value="0.24321" />
+        value="0.63096" />
       <inertia
-        ixx="0.00082645"
-        ixy="-2.6396E-05"
-        ixz="6.9353E-10"
-        iyy="0.00052575"
-        iyz="6.4571E-09"
-        izz="0.00052343" />
+        ixx="0.0015238"
+        ixy="1.7127E-09"
+        ixz="-6.387E-10"
+        iyy="0.0029312"
+        iyz="-3.3048E-09"
+        izz="0.0015238" />
     </inertial>
     <visual>
@@ -32,5 +32,5 @@
       <geometry>
         <mesh
-          filename="package://rover_description/meshes/STL/wheel/robot_wheel.stl" />
+          filename="package://rover_description/meshes/STL/wheel/wheel.STL" />
       </geometry>
       <material
@@ -46,5 +46,5 @@
       <geometry>
         <mesh
-          filename="package://rover_description/meshes/STL/wheel/robot_wheel.stl" />
+          filename="package://rover_description/meshes/STL/wheel/wheel.STL" />
       </geometry>
     </collision>

Commit message: gazebo simulation working

File: src/rover_description/robots/rover.urdf.xacro (robot description, xacro)
@@ -14,20 +14,20 @@
   <!-- Front Right Sus -->
   <xacro:steering_v0 prefix="front_right" parent="base_link">
-	<origin xyz="0.63104 -0.25952 -0.0205" rpy="0 0 0"/>
+	<origin xyz="0.63104 -0.25952 -0.0205" rpy="0 0 ${M_PI}"/>
 	<axis xyz="0 0 1"/>
   </xacro:steering_v0>
   <!-- Front Left Sus -->
   <xacro:steering_v0 prefix="front_left" parent="base_link">
-	<origin xyz="0.63104 0.25952 -0.0205" rpy="0 0 ${M_PI}"/>
+	<origin xyz="0.63104 0.25952 -0.0205" rpy="0 0 0"/>
 	<axis xyz="0 0 1"/>
   </xacro:steering_v0>
   <!-- Rear Right Sus -->
   <xacro:steering_v0 prefix="rear_right" parent="base_link">
-	<origin xyz="-0.63104 -0.25952 -0.0205" rpy="0 0 0"/>
+	<origin xyz="-0.63104 -0.25952 -0.0205" rpy="0 0 ${M_PI}"/>
 	<axis xyz="0 0 1"/>
   </xacro:steering_v0>
   <!-- Rear Left Sus -->
   <xacro:steering_v0 prefix="rear_left" parent="base_link">
-	<origin xyz="-0.63104 0.25952 -0.0205" rpy="0 0 ${M_PI}"/>
+	<origin xyz="-0.63104 0.25952 -0.0205" rpy="0 0 0"/>
 	<axis xyz="0 0 1"/>
   </xacro:steering_v0>
@@ -64,8 +64,8 @@
   <xacro:steering_trans_v0 prefix="rear_left"/>
   <!-- =============== Gazebo =============== -->
-  <!-- <gazebo>
+  <gazebo>
     <plugin name="gazebo_ros_control" filename="libgazebo_ros_control.so">
     </plugin>
-  </gazebo> -->
+  </gazebo>
   <!-- Base -->
   <xacro:base_gazebo_v0/>

File: src/rover_description/urdf/base/base.gazebo.xacro (robot description, xacro)
@@ -6,5 +6,5 @@
       <mu1 value="0.05" />
       <mu2 value="0.05" />
-      <material>Gazebo/Black</material>
+      <material>Gazebo/Grey</material>
     </gazebo>
   </xacro:macro>

File: src/rover_description/urdf/wheel/wheel.gazebo.xacro (robot description, xacro)
@@ -2,9 +2,9 @@
 <robot xmlns:xacro="http://ros.org/wiki/xacro">
   <xacro:macro name="wheel_gazebo_v0" params="prefix">
-  <gazebo reference="${prefix}_wheel_link">
-    <selfCollide>false</selfCollide>
+        <gazebo reference="${prefix}_wheel_link">
+          <selfCollide>false</selfCollide>
       <mu1 value="1.2" />
       <mu2 value="1.2" />
-      <material>Gazebo/Black</material>
+    <material>Gazebo/Black</material>
     </gazebo>
   </xacro:macro>

File: src/rover_description/urdf/wheel/wheel.urdf.xacro (robot description, xacro)
@@ -37,5 +37,5 @@
         name="">
         <color
-          rgba="0.25098 0.25098 0.25098 1" />
+          rgba="0.75294 0.75294 0.75294 1" />
       </material>
     </visual>

Commit message: New world

File: src/rover_description/robots/rover.urdf.xacro (robot description, xacro)
@@ -36,5 +36,5 @@
   <xacro:wheel_v0 prefix="ffr" parent="front_right_steering_link">
 	<origin xyz="0 0 -0.129" rpy="0 0 0"/>
-	<axis xyz="0 -1 0"/>
+	<axis xyz="0 1 0"/>
   </xacro:wheel_v0>
   <!--  Front Left Wheel -->
@@ -46,5 +46,5 @@
   <xacro:wheel_v0 prefix="rfr" parent="rear_right_steering_link">
 	<origin xyz="0 0 -0.129" rpy="0 0 0"/>
-	<axis xyz="0 -1 0"/>
+	<axis xyz="0 1 0"/>
   </xacro:wheel_v0>
   <!--  Rear Left Wheel -->

Commit message: add gps

File: src/rover_description/robots/rover.urdf.xacro (robot description, xacro)
@@ -63,7 +63,59 @@
   <xacro:steering_trans_v0 prefix="rear_right"/>
   <xacro:steering_trans_v0 prefix="rear_left"/>
+  <!-- =============== GPS Sensor =============== -->
+  <xacro:property name="gps_sensor_height" value="0.02" />
+  <xacro:property name="gps_sensor_width" value="0.02" />
+  <joint name="gps_joint" type="fixed">
+    <parent link="base_footprint"/>
+    <child link="gps_link"/>
+  </joint>
+  <link name="gps_link">
+    <collision>
+      <origin xyz="0 0 0.43" rpy="0 0 0"/>
+      <geometry>
+        <box size="${gps_sensor_width} ${gps_sensor_width} ${gps_sensor_height}"/>
+      </geometry>
+    </collision>
+    <visual>
+      <origin xyz="0 0 0.43" rpy="0 0 0"/>
+      <geometry>
+        <box size="${gps_sensor_width} ${gps_sensor_width} ${gps_sensor_height}"/>
+      </geometry>
+      <material name="orange"/>
+    </visual>
+    <inertial>
+      <origin xyz="0 0 0.43" rpy="0 0 0"/>
+      <mass value="1"/>
+      <inertia
+        ixx="1.0" ixy="0.0" ixz="0.0"
+        iyy="1.0" iyz="0.0"
+        izz="1.0"/>
+    </inertial>
+  </link>
+  <material name="orange">
+    <color rgba="${255/255} ${108/255} ${10/255} 1.0"/>
+  </material>
+  <gazebo reference="gps_link">
+    <material>Gazebo/Orange</material>
+  </gazebo>
   <!-- =============== Gazebo =============== -->
   <gazebo>
     <plugin name="gazebo_ros_control" filename="libgazebo_ros_control.so">
+    </plugin>
+    <plugin name="gazebo_ros_gps" filename="libhector_gazebo_ros_gps.so">
+        <updateRate>4.0</updateRate>
+        <bodyName>gps_link</bodyName>
+        <frameId>gps_link</frameId>
+        <topicName>/gps/fix</topicName>
+        <velocityTopicName>/gps/fix_velocity</velocityTopicName>
+        <referenceLatitude>-30.06022459407145675</referenceLatitude>
+        <referenceLongitude>-51.173913575780311191</referenceLongitude>
+        <referenceHeading>90</referenceHeading>
+        <referenceAltitude>10</referenceAltitude>
+        <offset>0 0 0</offset>
+        <drift>0.001 0.001 0.001</drift>
+        <gaussianNoise>0.05 0.05 0.05</gaussianNoise>
+        <velocityDrift>0.001 0.001 0.001</velocityDrift>
+        <velocityGaussianNoise>0.5 0.5 0.5</velocityGaussianNoise>
     </plugin>
   </gazebo>

Commit message: separate gps file

File: src/rover_description/robots/rover.urdf.xacro (robot description, xacro)
@@ -5,4 +5,5 @@
   <xacro:include filename="$(find rover_description)/urdf/suspension/suspension.urdf.xacro"/>
   <xacro:include filename="$(find rover_description)/urdf/wheel/wheel.urdf.xacro"/>
+  <xacro:include filename="$(find rover_description)/urdf/gps/gps.urdf.xacro"/>
   <!-- =============== Link & Joint =============== -->
   <!-- Base -->
@@ -63,40 +64,4 @@
   <xacro:steering_trans_v0 prefix="rear_right"/>
   <xacro:steering_trans_v0 prefix="rear_left"/>
-  <!-- =============== GPS Sensor =============== -->
-  <xacro:property name="gps_sensor_height" value="0.02" />
-  <xacro:property name="gps_sensor_width" value="0.02" />
-  <joint name="gps_joint" type="fixed">
-    <parent link="base_footprint"/>
-    <child link="gps_link"/>
-  </joint>
-  <link name="gps_link">
-    <collision>
-      <origin xyz="0 0 0.43" rpy="0 0 0"/>
-      <geometry>
-        <box size="${gps_sensor_width} ${gps_sensor_width} ${gps_sensor_height}"/>
-      </geometry>
-    </collision>
-    <visual>
-      <origin xyz="0 0 0.43" rpy="0 0 0"/>
-      <geometry>
-        <box size="${gps_sensor_width} ${gps_sensor_width} ${gps_sensor_height}"/>
-      </geometry>
-      <material name="orange"/>
-    </visual>
-    <inertial>
-      <origin xyz="0 0 0.43" rpy="0 0 0"/>
-      <mass value="1"/>
-      <inertia
-        ixx="1.0" ixy="0.0" ixz="0.0"
-        iyy="1.0" iyz="0.0"
-        izz="1.0"/>
-    </inertial>
-  </link>
-  <material name="orange">
-    <color rgba="${255/255} ${108/255} ${10/255} 1.0"/>
-  </material>
-  <gazebo reference="gps_link">
-    <material>Gazebo/Orange</material>
-  </gazebo>
   <!-- =============== Gazebo =============== -->
   <gazebo>

Commit message: fix wheel rotation issue

File: src/rover_description/robots/rover.urdf.xacro (robot description, xacro)
@@ -11,5 +11,5 @@
   <link name="base_footprint"/>
   <xacro:base_v0 parent="base_footprint">
-	<origin xyz="0 0 0.25" rpy="0 0 -1.570796"/>
+	<origin xyz="0 0 0.25" rpy="0 0 0"/>
   </xacro:base_v0>
   <!-- Suspension -->
@@ -38,20 +38,20 @@
   <xacro:wheel_v0 prefix="ffr" parent="front_right_steering_link">
 	<origin xyz="0 0 -0.129" rpy="0 0 0"/>
-	<axis xyz="0 1 0"/>
+	<axis xyz="0 -1 0"/>
   </xacro:wheel_v0>
   <!--  Front Left Wheel -->
   <xacro:wheel_v0 prefix="ffl" parent="front_left_steering_link">
 	<origin xyz="0 0 -0.129" rpy="0 0 0"/>
-	<axis xyz="0 -1 0"/>
+	<axis xyz="0 1 0"/>
   </xacro:wheel_v0>
   <!-- Rear Right Wheel -->
   <xacro:wheel_v0 prefix="rfr" parent="rear_right_steering_link">
 	<origin xyz="0 0 -0.129" rpy="0 0 0"/>
-	<axis xyz="0 1 0"/>
+	<axis xyz="0 -1 0"/>
   </xacro:wheel_v0>
   <!--  Rear Left Wheel -->
   <xacro:wheel_v0 prefix="rfl" parent="rear_left_steering_link">
 	<origin xyz="0 0 -0.129" rpy="0 0 0"/>
-	<axis xyz="0 -1 0"/>
+	<axis xyz="0 1 0"/>
   </xacro:wheel_v0>
   <!-- ===============  Wheel Transmission =============== -->
